File: mcu_power.kicad_sch (KiCad schematic)
At the start: 8 parts, among them U3 SiWG917Y

Commit message: added schematics comments of review 1
Parts:
- removed C30, C31: 1pF, Capacitor_SMD:C_0402_1005Metric, symbol #dzdb:g_cap/C-1p-0402
- added C49, C50: 1pF, Capacitor_SMD:C_0402_1005Metric, symbol #dzdb:g_cap/C-1p-0402
- added J9: U.FL, Connector_Coaxial:U.FL_Hirose_U.FL-R-SMT-1_Vertical, symbol #dzdb:s_mech/M-TEC-CONUFL001-SMD-T
Connections:
- net GND: now also L3.1, C49.1, C50.1, J9.2 (Ext)
- net at U3.10 (RF): now also L3.2, J9.1 (In); no longer L3.1
- net at U3.1 (ANT_TUNE_1): now also C50.2
- net at U3.61 (ANT_TUNE_2): now also C49.2
- no-connect marks 5 -> 2
Other:
- moved on the sheet: L3

Commit message: changes after first review: add lvl shifters, board at 1v8, new power tree
Connections:
- net VIO: no longer C12.1, C13.1, U3.34 (VBATT)
- new net 3V3_VBUS: C12.1, C13.1, U3.34 (VBATT)
Changed lines of the file:
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@@
 		(fill
 			(type color)
-			(color 255 153 0 1)
+			(color 255 253 31 1)
 		)
 		(effects
@@
 		(fill
 			(type color)
-			(color 255 153 0 1)
+			(color 255 252 69 1)
 		)
 		(effects
@@
 	)
 	(symbol
+		(lib_id "power:+BATT")
+		(at 34.29 54.61 0)
+		(unit 1)
+		(body_style 1)
+		(exclude_from_sim no)
+		(in_bom yes)
+		(on_board yes)
+		(in_pos_files yes)
+		(dnp no)
+		(property "Reference" "#PWR0121"
+			(at 34.29 58.42 0)
+			(hide yes)
+			(show_name no)
+			(do_not_autoplace no)
+			(effects
+				(font
+					(size 1.27 1.27)
+				)
+			)
+		)
+		(property "Value" "3V3_VBUS"
+			(at 29.972 50.546 0)
+			(show_name no)
+			(do_not_autoplace no)
+			(effects
+				(font
+					(size 1.27 1.27)
+				)
+				(justify left)
+			)
+		)
+		(property "Footprint" ""
+			(at 34.29 54.61 0)
+			(hide yes)
+			(show_name no)
+			(do_not_autoplace no)
+			(effects
+				(font
+					(size 1.27 1.27)
+				)
+			)
+		)
+		(property "Datasheet" ""
+			(at 34.29 54.61 0)
+			(hide yes)
+			(show_name no)
+			(do_not_autoplace no)
+			(effects
+				(font
+					(size 1.27 1.27)
+				)
+			)
+		)
+		(property "Description" "Power symbol creates a global label with name \"+BATT\""
+			(at 34.29 54.61 0)
+			(hide yes)
+			(show_name no)
+			(do_not_autoplace no)
+			(effects
+				(font
+					(size 1.27 1.27)
+				)
+			)
+		)
+		(pin "1"
+		)
+		(instances
+			(project "wius_new"
+				(path "/8543d6cf-82a6-4fc5-8760-a0773a1d6e4c/93f533c5-fe26-4cf1-a6b2-37346d84bc0c/d5bbc3da-8f67-4e14-ac58-596682e02652"
+					(reference "#PWR0121")
+					(unit 1)
+				)
+			)
+		)
+	)
+	(symbol
 		(lib_id "#dzdb:g_cap/C-1u-0402")
 		(at 34.29 63.5 0)
@@
 					(unit 1)
 				)
-			)
-		)
-	)
-	(symbol
-		(lib_id "power:+3V3")
-		(at 34.29 54.61 0)
-		(unit 1)
-		(body_style 1)
-		(exclude_from_sim no)
-		(in_bom yes)
-		(on_board yes)
-		(in_pos_files yes)
-		(dnp no)
-		(fields_autoplaced yes)
-		(property "Reference" "#PWR040"
-			(at 34.29 58.42 0)
-			(hide yes)
-			(show_name no)
-			(do_not_autoplace no)
-			(effects
-				(font
-					(size 1.27 1.27)
-				)
-			)
-		)
-		(property "Value" "VIO"
-			(at 36.83 53.3399 0)
-			(show_name no)
-			(do_not_autoplace no)
-			(effects
-				(font
-					(size 1.27 1.27)
-				)
-				(justify left)
-			)
-		)
-		(property "Footprint" ""
-			(at 34.29 54.61 0)
-			(hide yes)
-			(show_name no)
-			(do_not_autoplace no)
-			(effects
-				(font
-					(size 1.27 1.27)
-				)
-			)
-		)
-		(property "Datasheet" ""
-			(at 34.29 54.61 0)
-			(hide yes)
-			(show_name no)
-			(do_not_autoplace no)
-			(effects
-				(font
-					(size 1.27 1.27)
-				)
-			)
-		)
-		(property "Description" "Power symbol creates a global label with name \"+3V3\""
-			(at 34.29 54.61 0)
-			(hide yes)
-			(show_name no)
-			(do_not_autoplace no)
-			(effects
-				(font
-					(size 1.27 1.27)
-				)
-			)
-		)
-		(pin "1"
-		)
-		(instances
-			(project "wius_new"
-				(path "/8543d6cf-82a6-4fc5-8760-a0773a1d6e4c/93f533c5-fe26-4cf1-a6b2-37346d84bc0c/d5bbc3da-8f67-4e14-ac58-596682e02652"
-					(reference "#PWR040")
-					(unit 1)
-				)
