File: mcu_power.kicad_sch (KiCad schematic)
At the start: 9 parts, among them J9 U.FL, U3 SiWG917Y

Commit message: Add comments from layout meeting 20.07.2026
Connections:
- net 1V8 is gone; now on net Flash_IO_VDD: C24.1, U3.54 (FLASH_IO_VDD)
- net Flash_IO_VDD: now reaches U3.36 (1V8_LDO)
- no-connect marks 2 -> 1
Other:
- moved on the sheet: C14, C24
