File: power_conv.kicad_sch (KiCad schematic)
At the start: 20 parts, among them IC1 BQ24040DSQT, U1 TPS62840YBGR

Commit message: updated routing SPI, change 0402 to 0201
Parts:
- removed C4, C5: 100nF, Capacitor_SMD:C_0402_1005Metric, symbol #dzdb:g_cap/C-100n-0402
- added C39, C40: 100nF, Capacitor_SMD:C_0201_0603Metric, symbol #dzdb:g_cap/C-100n-0201
Connections:
- net BATT_SENSE: now also C40.1
- net GND: now also C39.2, C40.2
- net at R3.2, U1.C1 (EN): now also C39.1
