File: Peripherals.kicad_sch (KiCad schematic)
At the start: 23 parts, among them J3 1040310811, U5 LSM6DSV, U8 SN74AXC4T774RSVR

Commit message: updated routing
Connections:
- net GND: now also U8.5 (DIR3); no longer U8.15 (DIR1)
- net SPI_MCU.SCK: now also U8.1 (A1); no longer U8.3 (A3)
- net SPI_SD.MISO: now also U8.10 (B3); no longer U8.12 (B1)
- net VIO: now also U8.15 (DIR1); no longer U8.5 (DIR3)
- net at R49.1: now also U8.12 (B1); no longer U8.10 (B3)
- net at R47.2: now also U8.3 (A3); no longer U8.1 (A1)
Other:
- moved on the sheet: R47, R49
