File: mcu_io.kicad_sch (KiCad schematic)
At the start: 14 parts, among them U3 SiWG917Y, U9 PCAL6408AHK

Commit message: updated eeprom and oscillator
Connections:
- net INT_SD: now also U3.43 (GPIO_51); no longer U9.9 (P6)
Changed lines of the file:
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@@
+	)
+	(no_connect
+		(at 227.33 78.74)
 	)
 	(no_connect
@@
 	)
 	(no_connect
-		(at 96.52 101.6)
-	)
-	(no_connect
 		(at 55.88 96.52)
 	)
@@
 	(wire
 		(pts
-			(xy 236.22 78.74) (xy 227.33 78.74)
+			(xy 105.41 101.6) (xy 96.52 101.6)
 		)
 		(stroke
@@
 	(hierarchical_label "INT_SD"
 		(shape bidirectional)
-		(at 236.22 78.74 0)
-		(effects
-			(font
+		(at 105.41 101.6 0)
+		(effects
+			(font
